File: hardware/trhmsx_v1.0/trhmsx/trhmsx.kicad_sch (KiCad schematic)
At the start: 81 parts, among them J1 Micro_SD_Card_Det1, J10 USB_A, J13 Mini-DIN-6, J2 RCA, J3 DH15, J4 Barrel_Jack, J5 Conn_01x02, J6 Conn_01x05, J7 Conn_02x25_Odd_Even, J8 Conn_02x25_Odd_Even, J9 AudioJack2_Ground, SW1 SW_Push, SW2 SW_DIP_x08, U1 EP1C12Q240C8N, U2 AMS1117-1.5, U3 AMS1117-3.3, U4 M51953BFP, U5 NC7WZU04P6X, U6 4053, Y1 Crystal

Commit message: Joysticks, memory and active serial config
Parts:
- removed C18, C19, C20: 220uF, symbol Device:C_Polarized
- removed C4, C5, C7, C8: 100nF, symbol Device:C_Polarized
- removed U6: 4053, symbol 4xxx:4053
- added C18, C19, C20, C21, C22, C4, C5, C7, C8: 0.1uF, symbol Device:C
- added IC1: EPCS4, EPCS4:SO08, symbol TRHMSX:EPCS4
- added J11: JOY1, symbol Connector:DE9_Plug
- added J12: JOY2, symbol Connector:DE9_Plug
- added J14: Conn_02x05_Odd_Even, symbol Connector_Generic:Conn_02x05_Odd_Even
- added RN24, RN25, RN26, RN27, RN28: 10K, symbol Device:R_Pack04_Split
- added U6: MT48LC16M16A2TG, Package_SO:TSOP-II-54_22.2x10.16mm_P0.8mm, symbol Memory_RAM:MT48LC16M16A2TG
- Y1: value Crystal -> 21.47727 MHz
Connections:
- net +1V5: now also U1.103 (VCCINT_4), U1.110 (VCCINT_3), U1.72 (VCCINT), U1.81 (VCCINT_5), U1.90 (VCCINT), U1.97 (VCCINT_2), C5.1
- net +3.3V: now also U1.112 (VCCIO4), U1.130 (VCCIO3_2), U1.157 (VCCIO3), U1.22 (VCCIO1_2), U1.51 (VCCIO1_3), U1.70 (VCCIO4), U1.9 (VCCIO1), U1.92 (VCCIO4_2), C18.1, C19.1, C20.2, C22.1, C8.1, IC1.3 (VCC@3), IC1.7 (VCC@7), IC1.8 (VCC@8), J14.4 (Pin_4), RN24.5 (R4.2), RN24.6 (R3.2), RN24.7 (R2.2), RN24.8 (R1.2), RN25.6 (R3.2), RN25.7 (R2.2), RN25.8 (R1.2), RN26.6 (R3.2), RN26.7 (R2.2), RN26.8 (R1.2), RN27.5 (R4.2), RN27.6 (R3.2), RN27.7 (R2.2), RN27.8 (R1.2), RN28.1 (R1.1), RN28.2 (R2.1), RN28.3 (R3.1), U6.1 (VDD), U6.14 (VDD), U6.27 (VDD), U6.3 (VDDQ), U6.43 (VDDQ), U6.49 (VDDQ), U6.9 (VDDQ)
- net +5V: now also C21.1, C4.1, C7.1, J11.5, J12.5
- net GND: now also C18.2, C19.2, C20.1, C21.2, C4.2, C5.2, C7.2, C8.2, IC1.4 (GND), J11.9, J12.9, J14.10 (Pin_10), J14.2 (Pin_2), RN28.4 (R4.1), U6.12 (VSSQ), U6.28 (VSS), U6.41 (VSS), U6.46 (VSSQ), U6.52 (VSSQ), U6.54 (VSS), U6.6 (VSSQ)
- net VB_CV: now also J3.3
- net VG_SY: now also J3.2
- net VR_SC: now also J3.1
- net ~{RESET}: no longer J7.15 (Pin_15), J8.15 (Pin_15), RN3.1 (R1.1)
- net at C2.1, R5.1, U5.1 (A1)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: now also C22.2
- net VBO: no longer names the net of C15.1, RN14.1 (R1.1), RN15.8 (R1.2)
- net VGO: no longer names the net of C16.1, RN16.3 (R3.1), RN17.6 (R3.2)
- net VRO: no longer names the net of C17.1, RN20.1 (R1.1), RN21.8 (R1.2)
- net ~{BUSDIR} renamed BUSDIR
- net ~{CS12} renamed CS12
- net ~{CS1} renamed CS1
- net ~{CS2} renamed CS2
- net ~{INT} renamed INT
- net ~{IORQ} renamed IORQ
- net ~{M1} renamed M1
- net ~{MERQ} renamed MERQ
- net ~{RD} renamed RD
- net ~{RFSH} renamed RFSH
- net ~{SLTSL} renamed SLTSL1
- net SLTSL1: no longer J7.4 (Pin_4)
- net ~{WAIT} renamed WAIT
- net ~{WR} renamed WR
- new net AS_CK: IC1.6 (DCLK), J14.1 (Pin_1)
- new net AS_CS: IC1.1 (NCS), J14.8 (Pin_8)
- new net AS_DI: IC1.2 (DATA), J14.7 (Pin_7)
- new net AS_DO: IC1.5 (ASDI), J14.9 (Pin_9)
- new net C_CE: J14.6 (Pin_6), RN28.5 (R4.2)
- new net C_CONF: J14.5 (Pin_5), RN28.7 (R2.2)
- new net C_DONE: J14.3 (Pin_3), RN28.8 (R1.2)
- new net C_STAT: RN28.6 (R3.2)
- new net IO0: J11.1, RN24.1 (R1.1)
- new net IO1: J11.6, RN24.2 (R2.1)
- new net IO10: J12.7, RN27.4 (R4.1)
- new net IO11: J12.3, RN26.1 (R1.1)
- new net IO12: J12.8, RN26.2 (R2.1)
- new net IO13: J12.4, RN26.3 (R3.1)
- new net IO2: J11.2, RN24.3 (R3.1)
- new net IO3: J11.7, RN24.4 (R4.1)
- new net IO4: J11.3, RN25.1 (R1.1)
- new net IO5: J11.8, RN25.2 (R2.1)
- new net IO6: J11.4, RN25.3 (R3.1)
- new net IO7: J12.1, RN27.1 (R1.1)
- new net IO8: J12.6, RN27.2 (R2.1)
- new net IO9: J12.2, RN27.3 (R3.1)
- new net MA0: U6.23 (A0)
- new net MA1: U6.24 (A1)
- new net MA10: U6.22 (A10)
- new net MA11: U6.35 (A11)
- new net MA12: U6.36 (A12)
- new net MA2: U6.25 (A2)
- new net MA3: U6.26 (A3)
- new net MA4: U6.29 (A4)
- new net MA5: U6.30 (A5)
- new net MA6: U6.31 (A6)
- new net MA7: U6.32 (A7)
- new net MA8: U6.33 (A8)
- new net MA9: U6.34 (A9)
- new net MBA0: U6.20 (BA0)
- new net MBA1: U6.21 (BA1)
- new net MCAS: U6.17 (~{CAS})
- new net MCKE: U6.37 (CKE)
- new net MCLK: U6.38 (CLK)
- new net MCS: U6.19 (~{CS})
- new net MD0: U6.2 (DQ0)
- new net MD1: U6.4 (DQ1)
- new net MD10: U6.45 (DQ10)
- new net MD11: U6.47 (DQ11)
- new net MD12: U6.48 (DQ12)
- new net MD13: U6.50 (DQ13)
- new net MD14: U6.51 (DQ14)
- new net MD15: U6.53 (DQ15)
- new net MD2: U6.5 (DQ2)
- new net MD3: U6.7 (DQ3)
- new net MD4: U6.8 (DQ4)
- new net MD5: U6.10 (DQ5)
- new net MD6: U6.11 (DQ6)
- new net MD7: U6.13 (DQ7)
- new net MD8: U6.42 (DQ8)
- new net MD9: U6.44 (DQ9)
- new net MLDQ: U6.15 (DQML)
- new net MRAS: U6.18 (~{RAS})
- new net MUDQ: U6.39 (DQMH)
- new net MWE: U6.16 (~{WE})
- new net RESET: J7.15 (Pin_15), J8.15 (Pin_15), RN3.1 (R1.1)
- new net SLTSL2: J7.4 (Pin_4)
- no-connect marks 13 -> 17
Other:
- moved on the sheet: C1, C12, C2, C3, C6, C9, D1, D2, D3, D4, D5, D6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

Commit message: finishing FPGA wiring
Parts:
- added C10, C6: 0.1uF, symbol Device:C
- added J8: EXPANSION, symbol Connector_Generic:Conn_02x25_Odd_Even
- added R11: 22, symbol Device:R
- added R6, R9: 10, symbol Device:R
- added RN1, RN10, RN11, RN13, RN14, RN15, RN16, RN2, RN25, RN3, RN4, RN5, RN6, RN7, RN8, RN9: 100, symbol Device:R_Pack04_Split
- J12: renamed from J7; value Conn_02x25_Odd_Even -> CART2
- J15: renamed from J8; value Conn_02x25_Odd_Even -> CART1
- R7: value 100R -> 100
- R8: renamed from R6; value 100R -> 100
- renumbered C22 to C11, C20 to C12, C3 to C13, C2 to C14, C19 to C15, C21 to C16, C12 to C17, C10 to C18, C11 to C19, C4 to C2, C13 to C20, C14 to C21, C15 to C22, C16 to C23, C17 to C24, C5 to C3, C6 to C4, C7 to C5, C8 to C7, C9 to C8, C18 to C9, J6 to J1, J9 to J10, J2 to J11, J3 to J13, J11 to J14, J4 to J2, J1 to J3, J5 to J4, J10 to J5, J13 to J6, J14 to J7, J12 to J9, R5 to R10, R11 to R3, R8 to R4, R12 to R5, RN28 to RN12, RN4 to RN19, RN5 to RN20, RN6 to RN21, RN7 to RN22, RN1 to RN23, RN2 to RN24, RN3 to RN26, RN26 to RN27, RN27 to RN28, RN8 to RN29, RN10 to RN30, RN12 to RN31, RN14 to RN32, RN16 to RN33, RN18 to RN34, RN20 to RN35, RN22 to RN36, RN25 to RN37, RN9 to RN38, RN11 to RN39, RN13 to RN40, RN15 to RN41, RN17 to RN42, RN19 to RN43, RN21 to RN44, RN23 to RN45, RN24 to RN46, SW2 to SW1, SW1 to SW2, U5 to U4, U6 to U5, U4 to U6
Connections:
- net ~{RESET} is gone; now on net RESET: U6.6 (OUT)
- net +12V: now also J8.48 (Pin_48)
- net +1V5: now also U1.191 (VCCINT_2), U1.198 (VCCINT_3), U1.204 (VCCINT_4), U1.211 (VCCINT_5), U1.220 (VCCINT_6), U1.229 (VCCINT), R6.2, R9.2
- net +3.3V: now also U1.148 (TMS), U1.155 (TDI), U1.172 (VCCIO3), U1.189 (VCCIO2), U1.209 (VCCIO2_2), U1.231 (VCCIO2_3)
- net +5V: now also J8.45 (Pin_45), J8.47 (Pin_47)
- net -12V: now also J8.50 (Pin_50)
- net A0: now also J8.28 (Pin_28), RN2.2 (R2.1)
- net A1: now also J8.27 (Pin_27), RN2.1 (R1.1)
- net A10: now also J8.20 (Pin_20), RN11.4 (R4.1)
- net A11: now also J8.19 (Pin_19), RN11.3 (R3.1)
- net A12: now also J8.23 (Pin_23), RN1.1 (R1.1)
- net A13: now also J8.26 (Pin_26), RN1.4 (R4.1)
- net A14: now also J8.25 (Pin_25), RN1.3 (R3.1)
- net A15: now also J8.18 (Pin_18), RN11.2 (R2.1)
- net A2: now also J8.30 (Pin_30), RN2.4 (R4.1)
- net A3: now also J8.29 (Pin_29), RN2.3 (R3.1)
- net A4: now also J8.32 (Pin_32), RN3.2 (R2.1)
- net A5: now also J8.31 (Pin_31), RN3.1 (R1.1)
- net A6: now also J8.22 (Pin_22), RN6.4 (R4.1)
- net A7: now also J8.21 (Pin_21), RN6.3 (R3.1)
- net A8: now also J8.24 (Pin_24), RN1.2 (R2.1)
- net A9: now also J8.17 (Pin_17), RN11.1 (R1.1)
- net AS_CK: now also U1.36 (DCLK)
- net AS_CS: now also U1.24 (IO_22)
- net AS_DI: now also U1.25 (DATA0)
- net AS_DO: now also U1.37 (IO_23)
- net CLK21M: now also U1.28 (CLK0)
- net CLOCK: now also J8.42 (Pin_42), RN6.2 (R2.1)
- net CS1: now also J8.1 (Pin_1), RN7.2 (R2.1)
- net CS12: now also J8.3 (Pin_3), RN7.4 (R4.1)
- net CS2: now also J8.2 (Pin_2), RN7.3 (R3.1)
- net C_CE: now also U1.33 (NCE)
- net C_CONF: now also U1.26 (NCONFIG)
- net C_DONE: now also U1.145 (CONF_DONE)
- net C_STAT: now also U1.146 (NSTATUS)
- net D0: now also J8.34 (Pin_34), RN3.4 (R4.1)
- net D1: now also J8.33 (Pin_33), RN3.3 (R3.1)
- net D2: now also J8.36 (Pin_36), RN4.2 (R2.1)
- net D3: now also J8.35 (Pin_35), RN4.1 (R1.1)
- net D4: now also J8.38 (Pin_38), RN4.4 (R4.1)
- net D5: now also J8.37 (Pin_37), RN4.3 (R3.1)
- net D6: now also J8.40 (Pin_40), RN5.2 (R2.1)
- net D7: now also J8.39 (Pin_39), RN5.1 (R1.1)
- net EXTCLK: now also U1.29 (CLK1)
- net GND: now also U1.10 (GND_3), U1.102 (GND_6), U1.109 (GND_7), U1.111 (GND_8), U1.129 (GND), U1.142 (GND_3), U1.147 (TCK), U1.150 (GNDG_PLL2), U1.151 (GNDA_PLL2), U1.171 (GND_2), U1.190 (GND_4), U1.192 (GND_3), U1.199 (GND_5), U1.205 (GND_6), U1.210 (GND_8), U1.212 (GND), U1.221 (GND_9), U1.230 (GND_7), U1.232 (GND_10), U1.30 (GNDA_PLL1), U1.31 (GNDG_PLL1), U1.34 (MSEL0), U1.35 (MSEL1), U1.40 (GND_4), U1.52 (GND_5), U1.69 (GND_6), U1.71 (GND), U1.80 (GND_2), U1.89 (GND_2), U1.91 (GND_4), U1.96 (GND_5), C10.2, C6.2, J8.41 (Pin_41), J8.43 (Pin_43)
- net HSYNC: now also RN25.3 (R3.1)
- net INT: now also J8.8 (Pin_8), RN9.1 (R1.1)
- net IO0: now also RN13.1 (R1.1)
- net IO1: now also RN13.2 (R2.1)
- net IO10: now also RN15.3 (R3.1)
- net IO11: now also RN15.4 (R4.1)
- net IO12: now also RN16.1 (R1.1)
- net IO13: now also RN16.2 (R2.1)
- net IO2: now also RN13.3 (R3.1)
- net IO3: now also RN13.4 (R4.1)
- net IO4: now also RN14.1 (R1.1)
- net IO5: now also RN14.2 (R2.1)
- net IO6: now also RN14.3 (R3.1)
- net IO7: now also RN14.4 (R4.1)
- net IO8: now also RN15.1 (R1.1)
- net IO9: now also RN15.2 (R2.1)
- net IORQ: now also J8.11 (Pin_11), RN9.4 (R4.1)
- net M1: now also J8.9 (Pin_9), RN9.2 (R2.1)
- net MA0: now also U1.203 (IO_36)
- net MA1: now also U1.206 (IO_37)
- net MA10: now also U1.202 (IO_35)
- net MA11: now also U1.225 (IO_50)
- net MA12: now also U1.224 (IO_49)
- net MA2: now also U1.207 (IO_38)
- net MA3: now also U1.208 (IO_39)
- net MA4: now also U1.235 (IO_56)
- net MA5: now also U1.234 (IO_55)
- net MA6: now also U1.233 (IO_54)
- net MA7: now also U1.228 (IO_53)
- net MA8: now also U1.227 (IO_52)
- net MA9: now also U1.226 (IO_51)
- net MBA0: now also U1.200 (IO_33)
- net MBA1: now also U1.201 (IO_34)
- net MCAS: now also U1.195 (IO_30)
- net MCKE: now also U1.39 (IO_25)
- net MCLK: now also R11.1
- net MCS: now also U1.197 (IO_32)
- net MD0: now also U1.181 (IO_20)
- net MD1: now also U1.182 (IO_21)
- net MD10: now also U1.218 (IO_45)
- net MD11: now also U1.217 (IO_44)
- net MD12: now also U1.216 (IO_43)
- net MD13: now also U1.215 (IO_42)
- net MD14: now also U1.214 (IO_41)
- net MD15: now also U1.213 (IO_40)
- net MD2: now also U1.183 (IO_22)
- net MD3: now also U1.184 (IO_23)
- net MD4: now also U1.185 (IO_24)
- net MD5: now also U1.186 (IO_25)
- net MD6: now also U1.187 (IO_26)
- net MD7: now also U1.188 (IO_27)
- net MD8: now also U1.222 (IO_47)
- net MD9: now also U1.219 (IO_46)
- net MERQ: now also J8.12 (Pin_12), RN10.1 (R1.1)
- net MLDQ: now also U1.193 (IO_28)
- net MRAS: now also U1.196 (IO_31)
- net MUDQ: now also U1.223 (IO_48)
- net MWE: now also U1.194 (IO_29)
- net PWRLED: now also U1.240 (IO)
- net RD: now also J8.14 (Pin_14), RN10.3 (R3.1)
- net RESET: now also J8.15 (Pin_15), RN6.1 (R1.1)
- net RFSH: now also J8.6 (Pin_6), RN8.3 (R3.1)
- net RSV16: now also J8.16 (Pin_16), RN10.4 (R4.1)
- net RSV5: now also J8.5 (Pin_5), RN8.2 (R2.1)
- net SCLK: now also RN25.4 (R4.1)
- net SDAT: now also RN25.1 (R1.1)
- net SL0: now also U1.105 (IO_17)
- net SL1: now also U1.106 (IO_18)
- net SL2: now also U1.107 (IO_19)
- net SL3: now also U1.108 (IO_20)
- net SL4: now also U1.113 (IO_21)
- net SL5: now also U1.114 (IO_22)
- net SLTSL1: now also J8.4 (Pin_4), RN8.1 (R1.1)
- net SLTSL2: now also RN7.1 (R1.1)
- net SOUND_L: now also J8.49 (Pin_49)
- net SR0: now also U1.115 (IO_23)
- net SR1: now also U1.116 (IO_24)
- net SR2: now also U1.117 (IO_25)
- net SR3: now also U1.118 (IO_26)
- net SR4: now also U1.119 (IO_27)
- net SR5: now also U1.120 (IO_28)
- net SW1: now also J8.44 (Pin_44), RN5.3 (R3.1)
- net SW2: now also J8.46 (Pin_46), RN5.4 (R4.1)
- net VB0: now also U1.77 (IO_56)
- net VB1: now also U1.78 (IO_57)
- net VB2: now also U1.79 (IO)
- net VB3: now also U1.82 (IO_2)
- net VB4: now also U1.83 (IO_3)
- net VB5: now also U1.84 (IO_4)
- net VG0: now also U1.85 (IO_5)
- net VG1: now also U1.86 (IO_6)
- net VG2: now also U1.87 (IO_7)
- net VG3: now also U1.88 (IO_8)
- net VG4: now also U1.93 (IO_9)
- net VG5: now also U1.94 (IO_10)
- net VR0: now also U1.95 (IO_11)
- net VR1: now also U1.98 (IO_12)
- net VR2: now also U1.99 (IO_13)
- net VR3: now also U1.100 (IO_14)
- net VR4: now also U1.101 (IO_15)
- net VR5: now also U1.104 (IO_16)
- net VSYNC: now also RN25.2 (R2.1)
- net WAIT: now also J8.7 (Pin_7), RN8.4 (R4.1)
- net WR: now also J8.13 (Pin_13), RN10.2 (R2.1)
- net at U1.161 (IO_2): now also RN1.6 (R3.2)
- net at U1.162 (IO_3): now also RN1.5 (R4.2)
- net at U1.163 (IO_4): now also RN2.8 (R1.2)
- net at U1.164 (IO_5): now also RN2.7 (R2.2)
- net at U1.165 (IO_6): now also RN2.6 (R3.2)
- net at U1.166 (IO_7): now also RN2.5 (R4.2)
- net at U1.167 (IO_8): now also RN3.8 (R1.2)
- net at U1.168 (IO_9): now also RN3.7 (R2.2)
- net at U1.169 (IO_10): now also RN3.6 (R3.2)
- net at U1.170 (IO_11): now also RN3.5 (R4.2)
- net at U1.173 (IO_12): now also RN4.8 (R1.2)
- net at U1.174 (IO_13): now also RN4.7 (R2.2)
- net at U1.175 (IO_14): now also RN4.6 (R3.2)
- net at U1.176 (IO_15): now also RN4.5 (R4.2)
- net at U1.177 (IO_16): now also RN5.8 (R1.2)
- net at U1.178 (IO_17): now also RN5.7 (R2.2)
- net at U1.179 (IO_18): now also RN5.6 (R3.2)
- net at U1.180 (IO_19): now also RN5.5 (R4.2)
- net USBN1: now reaches U1.236 (IO_57)
- net USBP1: now reaches U1.237 (IO_58)
- net USBN2: now reaches U1.238 (IO_59)
- net USBP2: now reaches U1.239 (IO_60)
- net at U1.1 (IO_2): now also RN13.8 (R1.2)
- net at U1.11 (IO_10): now also RN15.8 (R1.2)
- net at U1.12 (IO_11): now also RN15.7 (R2.2)
- net at U1.13 (IO_12): now also RN15.6 (R3.2)
- net at U1.14 (IO_13): now also RN15.5 (R4.2)
- net at U1.15 (IO_14): now also RN16.8 (R1.2)
- net at U1.16 (IO_15): now also RN16.7 (R2.2)
- net at U1.2 (IO_3): now also RN13.7 (R2.2)
- net at U1.27 (VCCA_PLL1): now also C10.1, R9.1
- net at U1.3 (IO_4): now also RN13.6 (R3.2)
- net at U1.38 (IO_24): now also R11.2
- net at U1.4 (IO_5): now also RN13.5 (R4.2)
- net at U1.5 (IO_6): now also RN14.8 (R1.2)
- net at U1.6 (IO_7): now also RN14.7 (R2.2)
- net at U1.7 (IO_8): now also RN14.6 (R3.2)
- net at U1.73 (IO_52): now also RN25.8 (R1.2)
- net at U1.74 (IO_53): now also RN25.7 (R2.2)
- net at U1.75 (IO_54): now also RN25.6 (R3.2)
- net at U1.76 (IO_55): now also RN25.5 (R4.2)
- net at U1.8 (IO_9): now also RN14.5 (R4.2)
- net at U1.121 (IO_29): now also RN7.8 (R1.2)
- net at U1.122 (IO_30): now also RN7.7 (R2.2)
- net at U1.123 (IO_31): now also RN7.6 (R3.2)
- net at U1.124 (IO_32): now also RN7.5 (R4.2)
- net at U1.125 (IO_33): now also RN8.8 (R1.2)
- net at U1.126 (IO_34): now also RN8.7 (R2.2)
- net at U1.127 (IO_35): now also RN8.6 (R3.2)
- net at U1.128 (IO_36): now also RN8.5 (R4.2)
- net at U1.131 (IO_37): now also RN9.8 (R1.2)
- net at U1.132 (IO_38): now also RN9.7 (R2.2)
- net at U1.133 (IO_39): now also RN9.6 (R3.2)
- net at U1.134 (IO_40): now also RN9.5 (R4.2)
- net at U1.135 (IO_41): now also RN10.8 (R1.2)
- net at U1.136 (IO_42): now also RN10.7 (R2.2)
- net at U1.137 (IO_43): now also RN10.6 (R3.2)
- net at U1.138 (IO_44): now also RN10.5 (R4.2)
- net at U1.139 (IO_45): now also RN11.8 (R1.2)
- net at U1.140 (IO_46): now also RN11.7 (R2.2)
- net at U1.141 (IO_47): now also RN11.6 (R3.2)
- net at U1.143 (IO_48): now also RN11.5 (R4.2)
- net at U1.144 (IO_49): now also U1.152 (CLK3), RN6.7 (R2.2)
- net at U1.153 (CLK2): now also RN6.8 (R1.2)
- net at U1.154 (VCCA_PLL2): now also C6.1, R6.1
- net at U1.156 (IO_50): now also RN6.6 (R3.2)
- net at U1.158 (IO_51): now also RN6.5 (R4.2)
- net at U1.159 (IO_52): now also RN1.8 (R1.2)
- net at U1.160 (IO): now also RN1.7 (R2.2)
- net BUSDIR renamed BDIR
- net BDIR: now also J8.10 (Pin_10), RN9.3 (R3.1)
- no-connect marks 17 -> 31
Other:
- moved on the sheet: J10, RN19A, RN19B, RN19C, RN19D, RN20A, RN20B, RN20C, RN20D, RN21A, RN21B, RN21C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

Commit message: USB wiring
Parts:
- added J2: USB EXPANSION, symbol Connector:USB_A
- added R10, R8: 1K, symbol Device:R
- added R4: 330, symbol Device:R
- added R6: 10K, symbol Device:R
- J6: renamed from J5; value USB_A -> KEYBOARD-USB
- J7: renamed from J6; value Mini-DIN-6 -> KEYBOARD-PS2
- R3: value 1K -> 330
- R5: value 1K -> 10K
- renumbered C6 to C4, C4 to C5, C5 to C6, J9 to J10, J10 to J11, J11 to J12, J12 to J13, J13 to J14, J14 to J15, J15 to J16, J2 to J3, J3 to J4, J4 to J5, J7 to J8, J8 to J9, R7 to R11, R8 to R12, R9 to R13, R10 to R14, R11 to R15, R6 to R7, R4 to R9, RN19 to RN17, RN20 to RN18, RN21 to RN19, RN22 to RN20, RN23 to RN21, RN24 to RN22, RN25 to RN23, RN26 to RN24, RN27 to RN25, RN28 to RN26, RN29 to RN27, RN30 to RN28, RN31 to RN29, RN32 to RN30, RN33 to RN31, RN34 to RN32, RN35 to RN33, RN36 to RN34, RN37 to RN35, RN38 to RN36, RN39 to RN37, RN40 to RN38, RN41 to RN39, RN42 to RN40, RN43 to RN41, RN44 to RN42, RN45 to RN43, RN46 to RN44
Connections:
- net +3.3V: now also R10.1, R8.1; no longer R3.1, R5.1
- net +5V: now also J2.1 (VBUS)
- net GND: now also R5.1, J2.4 (GND), J2.5 (Shield), R6.1
- net KCLK: now also R8.2; no longer R3.2
- net KDAT: now also R10.2; no longer R5.2
- net USBN1: now also R3.1
- net USBP1: now also R4.1
- net USBN2: no longer names the net of U1.238 (IO_59)
- net USBP2: no longer names the net of U1.239 (IO_60)
- new net: J2.2 (D-), R4.2, R6.2
- new net: J2.3 (D+), R3.2, R5.2
- no-connect marks 31 -> 34
Other:
- moved on the sheet: SW1

Commit message: First version of the PCB
Parts:
- removed J2: USB EXPANSION, symbol Connector:USB_A
- removed R3, R4: 330, symbol Device:R
- removed R5, R6: 10K, symbol Device:R
- added C16, C17, C18, C19, C20, C21, C22, C23: 0.1uF, Capacitor_SMD:C_0805_2012Metric, symbol Device:C
- added J2: ESP-01, Connector_PinSocket_2.54mm:PinSocket_2x04_P2.54mm_Vertical, symbol Connector_Generic:Conn_02x04_Odd_Even
- C1, C5, C8: footprint (none) -> Capacitor_SMD:CP_Elec_6.3x3
- C10, C11, C12, C13, C14, C15, C2, C6, C7, C9: footprint (none) -> Capacitor_SMD:C_0805_2012Metric
- C24: renamed from C16; footprint (none) -> Capacitor_SMD:C_0805_2012Metric
- C25: renamed from C17; footprint (none) -> Capacitor_SMD:C_0805_2012Metric
- C26: renamed from C18; footprint (none) -> Capacitor_SMD:C_0805_2012Metric
- C27: renamed from C19; footprint (none) -> Capacitor_SMD:C_0805_2012Metric
- C28: renamed from C20; footprint (none) -> Capacitor_SMD:CP_Elec_6.3x3
- C29: renamed from C21; footprint (none) -> Capacitor_SMD:CP_Elec_6.3x3
- C3: renamed from C4; footprint (none) -> Capacitor_SMD:C_0805_2012Metric
- C30: renamed from C22; footprint (none) -> Capacitor_SMD:CP_Elec_6.3x3
- C31: renamed from C23; footprint (none) -> Capacitor_SMD:CP_Elec_6.3x3
- C32: renamed from C24; footprint (none) -> Capacitor_SMD:CP_Elec_6.3x3
- C4: renamed from C3; footprint (none) -> Capacitor_SMD:C_0805_2012Metric
- D1, D2, D3, D4, D5, D6, D7, D8, D9: footprint (none) -> LED_SMD:LED_0805_2012Metric
- F1: footprint (none) -> Fuse:Fuse_1210_3225Metric
- IC1: footprint EPCS4:SO08 -> TRHMSX:SO08
- J1: value Conn_01x05 -> MODULE-12V; footprint (none) -> Connector_PinSocket_2.54mm:PinSocket_1x05_P2.54mm_Vertical
- J10, J15: footprint (none) -> Connector_Dsub:DSUB-9_Male_Horizontal_P2.77x2.84mm_EdgePinOffset4.94mm_Housed_MountingHolesOffset7.48mm
- J11: footprint (none) -> TRHMSX:PJ-307
- J12: footprint (none) -> TRHMSX:CUI_RCJ-044
- J13, J16: footprint (none) -> TRHMSX:TE_5530841-5
- J14: footprint (none) -> Connector_Dsub:DSUB-15-HD_Female_Horizontal_P2.29x1.98mm_EdgePinOffset3.03mm_Housed_MountingHolesOffset4.94mm
- J3: footprint (none) -> Connector_BarrelJack:BarrelJack_Horizontal
- J4: value Micro_SD_Card_Det1 -> MICRO-SD; footprint CRISAG:Conn_uSDcard -> TRHMSX:Conn_uSDcard
- J5: footprint (none) -> Connector_PinHeader_2.54mm:PinHeader_1x02_P2.54mm_Vertical
- J6: footprint (none) -> TRHMSX:TE_6364372-2
- J7: footprint (none) -> TRHMSX:TE_5749180-1
- J8: footprint (none) -> Connector_PinHeader_2.54mm:PinHeader_2x05_P2.54mm_Vertical
- J9: footprint (none) -> Connector_PinHeader_2.54mm:PinHeader_2x25_P2.54mm_Vertical
- R1, R2: footprint (none) -> Resistor_SMD:R_0805_2012Metric
- R10: renamed from R15; footprint (none) -> Resistor_SMD:R_0805_2012Metric
- R11: renamed from R14; footprint (none) -> Resistor_SMD:R_0805_2012Metric
- R3: renamed from R7; footprint (none) -> Resistor_SMD:R_0805_2012Metric
- R4: renamed from R8; footprint (none) -> Resistor_SMD:R_0805_2012Metric
- R5: renamed from R9; footprint (none) -> Resistor_SMD:R_0805_2012Metric
- R6: renamed from R10; footprint (none) -> Resistor_SMD:R_0805_2012Metric
- R7: renamed from R13; footprint (none) -> Resistor_SMD:R_0805_2012Metric
- R8: renamed from R11; footprint (none) -> Resistor_SMD:R_0805_2012Metric
- R9: renamed from R12; footprint (none) -> Resistor_SMD:R_0805_2012Metric
- RN1, RN10, RN11, RN12, RN13, RN14, RN15, RN16, RN17, RN18, RN19, RN2, RN20, RN21, RN22, RN23, RN24, RN25, RN26, RN27, RN28, RN29, RN3, RN30, RN31, RN32, RN33, RN34, RN35, RN36, RN37, RN38, RN39, RN4, RN40, RN41, RN42, RN43, RN44, RN5, RN6, RN7, RN8, RN9: footprint (none) -> Resistor_SMD:R_Array_Convex_4x0603
- SW1: footprint (none) -> Button_Switch_THT:SW_DIP_SPSTx08_Piano_10.8x21.88mm_W7.62mm_P2.54mm
- SW2: footprint (none) -> Button_Switch_THT:SW_Tactile_SPST_Angled_PTS645Vx83-2LFS
- U1: footprint QFP50P3460X3460X410-240N -> TRHMSX:QFP50P3460X3460X410-240N
- U4: footprint SOT65P210X110-6N -> TRHMSX:SOT65P210X110-6N
- U6: footprint (none) -> TRHMSX:SO08
- Y1: footprint (none) -> Crystal:Crystal_HC49-U_Vertical
Connections:
- net +1V5: now also C20.2, C21.2, C22.2, C23.2
- net +3.3V: now also RN24.1 (R1.1), RN24.2 (R2.1), RN24.3 (R3.1), RN24.4 (R4.1), C16.2, C17.2, C18.2, C19.2, J2.4 (Pin_4), J2.8 (Pin_8); no longer RN24.5 (R4.2), RN24.6 (R3.2), RN24.7 (R2.2), RN24.8 (R1.2)
- net GND: now also RN37.7 (R2.2), RN38.5 (R4.2), RN40.7 (R2.2), RN41.5 (R4.2), RN43.7 (R2.2), C16.1, C17.1, C18.1, C19.1, C20.1, C21.1, C22.1, C23.1, J2.1 (Pin_1); no longer RN37.2 (R2.1), RN38.4 (R4.1), RN40.2 (R2.1), RN41.4 (R4.1), RN43.2 (R2.1)
- net RESET: now also RN24.8 (R1.2); no longer RN24.1 (R1.1)
- net RFSH: now also RN24.5 (R4.2); no longer RN24.4 (R4.1)
- net RSV16: now also RN24.6 (R3.2); no longer RN24.3 (R3.1)
- net RSV5: now also RN24.7 (R2.2); no longer RN24.2 (R2.1)
- net SL0: now also RN29.4 (R4.1); no longer RN29.5 (R4.2)
- net SL1: now also RN29.3 (R3.1); no longer RN29.6 (R3.2)
- net SL2: now also RN29.2 (R2.1); no longer RN29.7 (R2.2)
- net SL3: now also RN29.1 (R1.1); no longer RN29.8 (R1.2)
- net SL4: now also RN28.4 (R4.1); no longer RN28.5 (R4.2)
- net SL5: now also RN28.3 (R3.1); no longer RN28.6 (R3.2)
- net SR0: now also RN28.2 (R2.1); no longer RN28.7 (R2.2)
- net SR1: now also RN28.1 (R1.1); no longer RN28.8 (R1.2)
- net SR2: now also RN27.4 (R4.1); no longer RN27.5 (R4.2)
- net SR3: now also RN27.3 (R3.1); no longer RN27.6 (R3.2)
- net SR4: now also RN27.2 (R2.1); no longer RN27.7 (R2.2)
- net SR5: now also RN27.1 (R1.1); no longer RN27.8 (R1.2)
- net USBN1: now also J2.2 (Pin_2)
- net USBP1: now also J2.7 (Pin_7)
- net VB0: now also RN31.2 (R2.1); no longer RN31.7 (R2.2)
- net VB1: now also RN31.1 (R1.1); no longer RN31.8 (R1.2)
- net VB2: now also RN30.4 (R4.1); no longer RN30.5 (R4.2)
- net VB3: now also RN30.3 (R3.1); no longer RN30.6 (R3.2)
- net VB4: now also RN30.2 (R2.1); no longer RN30.7 (R2.2)
- net VB5: now also RN30.1 (R1.1); no longer RN30.8 (R1.2)
- net VG0: now also RN32.4 (R4.1); no longer RN32.5 (R4.2)
- net VG1: now also RN32.3 (R3.1); no longer RN32.6 (R3.2)
- net VG2: now also RN32.2 (R2.1); no longer RN32.7 (R2.2)
- net VG3: now also RN32.1 (R1.1); no longer RN32.8 (R1.2)
- net VG4: now also RN31.4 (R4.1); no longer RN31.5 (R4.2)
- net VG5: now also RN31.3 (R3.1); no longer RN31.6 (R3.2)
- net VR0: now also RN34.2 (R2.1); no longer RN34.7 (R2.2)
- net VR1: now also RN34.1 (R1.1); no longer RN34.8 (R1.2)
- net VR2: now also RN33.4 (R4.1); no longer RN33.5 (R4.2)
- net VR3: now also RN33.3 (R3.1); no longer RN33.6 (R3.2)
- net VR4: now also RN33.2 (R2.1); no longer RN33.7 (R2.2)
- net VR5: now also RN33.1 (R1.1); no longer RN33.8 (R1.2)
- new net: RN30.7 (R2.2), RN39.2 (R2.1), RN39.8 (R1.2)
- new net: RN30.6 (R3.2), RN39.3 (R3.1), RN39.7 (R2.2)
- new net: RN33.7 (R2.2), RN42.2 (R2.1), RN42.8 (R1.2)
- new net: C31.1, RN31.6 (R3.2), RN40.3 (R3.1)
- new net: RN29.8 (R1.2), RN37.5 (R4.2), RN38.1 (R1.1)
- new net: RN29.7 (R2.2), RN38.2 (R2.1), RN38.8 (R1.2)
- new net: C32.1, RN33.8 (R1.2), RN42.1 (R1.1)
- new net: RN31.8 (R1.2), RN39.5 (R4.2), RN40.1 (R1.1)
- new net: RN31.7 (R2.2), RN40.2 (R2.1), RN40.8 (R1.2)
- new net: RN32.5 (R4.2), RN41.4 (R4.1), RN41.6 (R3.2)
- new net: C29.1, RN28.6 (R3.2), RN37.3 (R3.1)
- new net: RN32.8 (R1.2), RN40.5 (R4.2), RN41.1 (R1.1)
- new net: RN29.5 (R4.2), RN38.4 (R4.1), RN38.6 (R3.2)
- new net: C28.1, RN27.8 (R1.2), RN36.1 (R1.1)
- new net: RN30.5 (R4.2), RN39.4 (R4.1), RN39.6 (R3.2)
- new net: RN28.8 (R1.2), RN36.5 (R4.2), RN37.1 (R1.1)
- new net: RN33.6 (R3.2), RN42.3 (R3.1), RN42.7 (R2.2)
- new net: RN33.5 (R4.2), RN42.4 (R4.1), RN42.6 (R3.2)
- new net: C30.1, RN30.8 (R1.2), RN39.1 (R1.1)
- new net: RN32.6 (R3.2), RN41.3 (R3.1), RN41.7 (R2.2)
- new net: RN28.5 (R4.2), RN37.4 (R4.1), RN37.6 (R3.2)
- new net: RN34.8 (R1.2), RN42.5 (R4.2), RN43.1 (R1.1)
- new net: RN28.7 (R2.2), RN37.2 (R2.1), RN37.8 (R1.2)
- new net: RN27.7 (R2.2), RN36.2 (R2.1), RN36.8 (R1.2)
- new net: RN27.5 (R4.2), RN36.4 (R4.1), RN36.6 (R3.2)
- new net: RN34.7 (R2.2), RN43.2 (R2.1), RN43.8 (R1.2)
- new net: RN29.6 (R3.2), RN38.3 (R3.1), RN38.7 (R2.2)
- new net: RN27.6 (R3.2), RN36.3 (R3.1), RN36.7 (R2.2)
- new net: RN32.7 (R2.2), RN41.2 (R2.1), RN41.8 (R1.2)
- new net: RN31.5 (R4.2), RN40.4 (R4.1), RN40.6 (R3.2)
- no-connect marks 34 -> 36
Other:
- moved on the sheet: C10, C3, R10, R3, R7, RN10A, RN10B, RN10C, RN10D, RN11A, RN11B, RN11C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

Commit message: Initial placement
Parts:
- J9: now not fitted; now left out of the parts list
Changed lines of the file:
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@@
   (title_block
     (title "TRHMSX - The simple MSX2+ clone in FPGA")
-    (date "2023-08-27")
+    (date "2023-11-19")
     (rev "1.0")
     (company "The Retro Hacker")
@@
   )
   (symbol (lib_id "Connector_Generic:Conn_02x25_Odd_Even") (at 276.86 240.03 90) (unit 1)
-    (in_bom yes) (on_board yes) (dnp no) (fields_autoplaced)
+    (in_bom no) (on_board no) (dnp yes) (fields_autoplaced)
     (property "Reference" "J9" (at 243.84 237.49 90)
       (effects (font (size 1.27 1.27)) (justify left))
@@
       (effects (font (size 1.27 1.27)) hide)
     )
+    (property "Sim.Enable" "0" (at 276.86 240.03 0)
+      (effects (font (size 1.27 1.27)) hide)
+    )
