File: hardware/trhmsx/trhmsx.kicad_sch (KiCad schematic)
At the start: 124 parts, among them IC1 EPCS4, J1 MODULE-12V, J10 JOY2, J11 AudioJack2_Ground, J12 PJRAN1X1U02AUX, J13 CART2, J14 DH15, J15 JOY1, J16 CART1, J17 Conn_01x02, J2 ESP-01, J3 Barrel_Jack, J4 MICRO-SD, J5 Conn_01x02, J6 KEYBOARD-USB, J7 KEYBOARD-PS2, J8 Conn_02x05_Odd_Even, J9 EXPANSION, SW1 SW_DIP_x08, SW2 SW_Push, U1 EP1C12Q240C8N, U2 AMS1117-1.5, U3 AMS1117-3.3, U4 NC7WZU04P6X, U5 MT48LC16M16A2TG, U6 M51953BFP, Y1 21.47727 MHz

Commit message: 1.4 release. minor fixes.
Parts:
- J12: footprint TRHMSX:SWITCHCRAFT_PJRAN1X1U02AUX -> PJRAN1X1U02AUX:SWITCHCRAFT_PJRAN1X1U02AUX; Description_1 (none) -> RCA Phono Connectors RCA PHONO JACK WHT.
