File: hardware/1.5/trhmsx/trhmsx.kicad_sch (KiCad schematic)
At the start: 132 parts, among them J1 MODULE-12V, J10 JOY2, J11 AudioJack2_Ground, J12 Composite, J13 CART2, J14 DH15, J15 JOY1, J16 CART1, J17 Conn_01x02, J18 S-Video, J2 ESP-01, J3 Barrel_Jack, J4 MICRO-SD, J5 Conn_01x02, J6 KEYBOARD-USB, J7 KEYBOARD-PS2, J8 Conn_02x05_Odd_Even, J9 EXPANSION, SW1 SW_DIP_x08, SW2 SW_Push, SW3 SW_Push, U1 EP1C12Q240C8N, U2 AMS1117-1.5, U3 AMS1117-3.3, U4 NC7WZU04P6X, U5 MT48LC16M16A2TG, U6 M51953BFP, U7 CH559T, U8 EPCS4, Y1 21.47727 MHz

Commit message: Recompiling the firmware to support USB keyboards, fix for SVIDEO. 1.51 release.
Connections:
- net VG_SY: now also J18.3; no longer J18.4
- net VR_SC: now also J18.4; no longer J18.3
Changed lines of the file:
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@@
 	(title_block
 		(title "TRHMSX - A simple MSX2+ clone in FPGA")
-		(date "2024-11-10")
-		(rev "1.5")
+		(date "2024-12-31")
+		(rev "1.51")
 		(company "The Retro Hacker")
 		(comment 1 "Creative Commons Attribution-NonCommercial-ShareAlike 4.0 International License")
@@
 		)
 	)
+	(label "VR_SC"
+		(at 439.42 91.44 180)
+		(fields_autoplaced yes)
+		(effects
+			(font
+				(size 1.27 1.27)
+			)
+			(justify right bottom)
+		)
+	)
 	(label "IO9"
 		(at 345.44 60.96 0)
@@
 		)
 	)
-	(label "VR_SC"
-		(at 439.42 88.9 180)
-		(fields_autoplaced yes)
-		(effects
-			(font
-				(size 1.27 1.27)
-			)
-			(justify right bottom)
-		)
-	)
 	(label "MA2"
 		(at 107.95 129.54 0)
@@
 		)
 	)
-	(label "VG_SY"
-		(at 439.42 91.44 180)
-		(fields_autoplaced yes)
-		(effects
-			(font
-				(size 1.27 1.27)
-			)
-			(justify right bottom)
-		)
-	)
 	(label "SLTSL2"
 		(at 490.22 279.4 0)
@@
 		)
 	)
+	(label "VG_SY"
+		(at 439.42 88.9 180)
+		(fields_autoplaced yes)
+		(effects
+			(font
+				(size 1.27 1.27)
+			)
+			(justify right bottom)
+		)
+	)
 	(label "MD0"
 		(at 402.59 266.7 0)
@@
 		(at 553.72 365.76 0)
 		(unit 1)
-		(exclude_from_sim no)
+		(exclude_from_sim yes)
 		(in_bom no)
 		(on_board no)
@@
 			(at 553.72 365.76 0)
 			(effects
-				(font
-					(size 1.27 1.27)
-				)
-				(hide yes)
-			)
-		)
-		(property "Sim.Enable" "0"
-			(at 553.72 365.76 0)
-			(effects
